Commit message: edit params of waiteronix cong

File: waiteronix/urdf/waiteronix.xacro (robot description, xacro)
@@ -148,5 +148,5 @@
     type="continuous">
     <origin
-      xyz="-0.0087223 -0.224 0.054"
+      xyz="-0.0087223 -0.224 0.0538"
       rpy="0 0 0" />
     <parent
@@ -155,8 +155,5 @@
       link="Right_Wheel" />
     <axis
-      xyz="0 -1 0" />
-    <limit
-      effort="40"
-      velocity="10" />
+      xyz="0 1 0" />
   </joint>
   <link
@@ -204,5 +201,5 @@
     type="continuous">
     <origin
-      xyz="-0.0087223 0.224 0.054"
+      xyz="-0.0087223 0.224 0.0538"
       rpy="0 0 0" />
     <parent
@@ -211,8 +208,5 @@
       link="Left_Wheel" />
     <axis
-      xyz="0 -1 0" />
-    <limit
-      effort="40"
-      velocity="10" />
+      xyz="0 1 0" />
   </joint>
   <link

Commit message: adding caster wheel reference to waiteronix.gazebo and changing caster wheels to fixed again

File: waiteronix/urdf/waiteronix.xacro (robot description, xacro)
@@ -5,4 +5,7 @@
      For more information, please see http://wiki.ros.org/sw_urdf_exporter -->
   <xacro:include filename="$(find waiteronix)/urdf/waiteronix.gazebo"/>
+  <xacro:include filename="$(find waiteronix)/urdf/caster_wheels.xacro"/>
+  <xacro:include filename="$(find waiteronix)/urdf/diff_wheels.xacro"/>
+  <xacro:include filename="$(find waiteronix)/urdf/sensors.xacro"/>
   <link name="robot_footprint">
   </link>
@@ -104,486 +107,3 @@
       xyz="0 0 0" />
   </joint>
-  <link
-    name="Right_Wheel">
-    <inertial>
-      <origin
-        xyz="2.5996E-07 0.037854 6.57E-06"
-        rpy="0 0 0" />
-      <mass
-        value="1.21" />
-      <inertia
-        ixx="0.0022228"
-        ixy="-1.8762E-08"
-        ixz="1.5736E-09"
-        iyy="0.0036326"
-        iyz="-4.7418E-07"
-        izz="0.0022228" />
-    </inertial>
-    <visual>
-      <origin
-        xyz="0 0 0"
-        rpy="0 0 0" />
-      <geometry>
-        <mesh
-          filename="package://waiteronix/meshes/Right_Wheel.STL" />
-      </geometry>
-      <material
-        name="">
-        <color
-          rgba="0.75294 0.75294 0.75294 1" />
-      </material>
-    </visual>
-    <collision>
-      <origin
-        xyz="0 0 0"
-        rpy="0 0 0" />
-      <geometry>
-        <mesh
-          filename="package://waiteronix/meshes/Right_Wheel.STL" />
-      </geometry>
-    </collision>
-  </link>
-  <joint
-    name="Right_Wheel_Joint"
-    type="continuous">
-    <origin
-      xyz="-0.0087223 -0.224 0.038"
-      rpy="0 0 0" />
-    <parent
-      link="base_link" />
-    <child
-      link="Right_Wheel" />
-    <axis
-      xyz="0 1 0" />
-    <limit
-      effort="40"
-      velocity="10" />
-  </joint>
-  <link
-    name="Left_Wheel">
-    <inertial>
-      <origin
-        xyz="2.5996E-07 -0.037854 6.57E-06"
-        rpy="0 0 0" />
-      <mass
-        value="1.21" />
-      <inertia
-        ixx="0.0022228"
-        ixy="1.8762E-08"
-        ixz="1.5736E-09"
-        iyy="0.0036326"
-        iyz="4.7418E-07"
-        izz="0.0022228" />
-    </inertial>
-    <visual>
-      <origin
-        xyz="0 0 0"
-        rpy="0 0 0" />
-      <geometry>
-        <mesh
-          filename="package://waiteronix/meshes/Left_Wheel.STL" />
-      </geometry>
-      <material
-        name="">
-        <color
-          rgba="0.75294 0.75294 0.75294 1" />
-      </material>
-    </visual>
-    <collision>
-      <origin
-        xyz="0 0 0"
-        rpy="0 0 0" />
-      <geometry>
-        <mesh
-          filename="package://waiteronix/meshes/Left_Wheel.STL" />
-      </geometry>
-    </collision>
-  </link>
-  <joint
-    name="Left_Wheel_Joint"
-    type="continuous">
-    <origin
-      xyz="-0.0087223 0.224 0.038"
-      rpy="0 0 0" />
-    <parent
-      link="base_link" />
-    <child
-      link="Left_Wheel" />
-    <axis
-      xyz="0 1 0" />
-    <limit
-      effort="40"
-      velocity="10" />
-  </joint>
-  <link
-    name="Camera">
-    <inertial>
-      <origin
-        xyz="-0.027769 0.064365 -0.00028163"
-        rpy="0 0 0" />
-      <mass
-        value="0.55893" />
-      <inertia
-        ixx="0.0029329"
-        ixy="-9.3578E-07"
-        ixz="8.9611E-08"
-        iyy="0.00023177"
-        iyz="-9.4508E-09"
-        izz="0.0030272" />
-    </inertial>
-    <visual>
-      <origin
-        xyz="0 0 0"
-        rpy="0 0 0" />
-      <geometry>
-        <mesh
-          filename="package://waiteronix/meshes/Camera.STL" />
-      </geometry>
-      <material
-        name="">
-        <color
-          rgba="0.49412 0.49412 0.49412 1" />
-      </material>
-    </visual>
-    <collision>
-      <origin
-        xyz="0 0 0"
-        rpy="0 0 0" />
-      <geometry>
-        <mesh
-          filename="package://waiteronix/meshes/Camera.STL" />
-      </geometry>
-    </collision>
-  </link>
-  <joint
-    name="Camera_Joint"
-    type="fixed">
-    <origin
-      xyz="0.24478 -0.064307 0.0965"
-      rpy="0 0 0" />
-    <parent
-      link="base_link" />
-    <child
-      link="Camera" />
-    <axis
-      xyz="1 0 0" />
-  </joint>
-  <link
-    name="Lidar">
-    <inertial>
-      <origin
-        xyz="8.3267E-17 -1.9976E-15 -0.013917"
-        rpy="0 0 0" />
-      <mass
-        value="0.12331" />
-      <inertia
-        ixx="8.5672E-05"
-        ixy="-3.3087E-22"
-        ixz="-3.3193E-19"
-        iyy="8.5672E-05"
-        iyz="-1.4388E-23"
-        izz="0.00010203" />
-    </inertial>
-    <visual>
-      <origin
-        xyz="0 0 0"
-        rpy="0 0 0" />
-      <geometry>
-        <mesh
-          filename="package://waiteronix/meshes/Lidar.STL" />
-      </geometry>
-      <material
-        name="">
-        <color
-          rgba="0 0.75294 0 1" />
-      </material>
-    </visual>
-    <collision>
-      <origin
-        xyz="0 0 0"
-        rpy="0 0 0" />
-      <geometry>
-        <mesh
-          filename="package://waiteronix/meshes/Lidar.STL" />
-      </geometry>
-    </collision>
-  </link>
-  <joint
-    name="Lidar_Joint"
-    type="fixed">
-    <origin
-      xyz="0.185 0 0.21663"
-      rpy="0 0 0" />
-    <parent
-      link="base_link" />
-    <child
-      link="Lidar" />
-    <axis
-      xyz="0 0 1" />
-  </joint>
-  <link
-    name="IMU">
-    <inertial>
-      <origin
-        xyz="-1.8518E-16 -6.2326E-15 -0.005"
-        rpy="0 0 0" />
-      <mass
-        value="0.0007854" />
-      <inertia
-        ixx="1.1454E-08"
-        ixy="1.831E-25"
-        ixz="-3.3736E-23"
-        iyy="1.1454E-08"
-        iyz="1.7323E-23"
-        izz="9.8175E-09" />
-    </inertial>
-    <visual>
-      <origin
-        xyz="0 0 0"
-        rpy="0 0 0" />
-      <geometry>
-        <mesh
-          filename="package://waiteronix/meshes/IMU.STL" />
-      </geometry>
-      <material
-        name="">
-        <color
-          rgba="0 0.75294 0 1" />
-      </material>
-    </visual>
-    <collision>
-      <origin
-        xyz="0 0 0"
-        rpy="0 0 0" />
-      <geometry>
-        <mesh
-          filename="package://waiteronix/meshes/IMU.STL" />
-      </geometry>
-    </collision>
-  </link>
-  <joint
-    name="IMU_Joint"
-    type="fixed">
-    <origin
-      xyz="0 0 0.289"
-      rpy="0 0 0" />
-    <parent
-      link="base_link" />
-    <child
-      link="IMU" />
-    <axis
-      xyz="0 0 1" />
-  </joint>
-  <link
-    name="F_W_Front_Left">
-    <inertial>
-      <origin
-        xyz="0.13868 0.123 -1.4438E-14"
-        rpy="0 0 0" />
-      <mass
-        value="0.059636" />
-      <inertia
-        ixx="1.6012E-05"
-        ixy="-1.927E-20"
-        ixz="-9.0002E-22"
-        iyy="2.7287E-05"
-        iyz="-2.1253E-20"
-        izz="1.6012E-05" />
-    </inertial>
-    <visual>
-      <origin
-        xyz="0 0 0"
-        rpy="0 0 0" />
-      <geometry>
-        <mesh
-          filename="package://waiteronix/meshes/F_W_Front_Left.STL" />
-      </geometry>
-      <material
-        name="">
-        <color
-          rgba="0.50196 0.50196 1 1" />
-      </material>
-    </visual>
-    <collision>
-      <origin
-        xyz="0 0 0"
-        rpy="0 0 0" />
-      <geometry>
-        <mesh
-          filename="package://waiteronix/meshes/F_W_Front_Left.STL" />
-      </geometry>
-    </collision>
-  </link>
-  <joint
-    name="F_W_Front_Left_Joint"
-    type="fixed">
-    <origin
-      xyz="0 0 0"
-      rpy="0 0 0" />
-    <parent
-      link="base_link" />
-    <child
-      link="F_W_Front_Left" />
-    <axis
-      xyz="0 1 0" />
-  </joint>
-  <link
-    name="F_W_Front_Right">
-    <inertial>
-      <origin
-        xyz="0.13868 -0.123 2.4819E-14"
-        rpy="0 0 0" />
-      <mass
-        value="0.059636" />
-      <inertia
-        ixx="1.6012E-05"
-        ixy="5.4827E-21"
-        ixz="-3.2336E-22"
-        iyy="2.7287E-05"
-        iyz="-3.8765E-20"
-        izz="1.6012E-05" />
-    </inertial>
-    <visual>
-      <origin
-        xyz="0 0 0"
-        rpy="0 0 0" />
-      <geometry>
-        <mesh
-          filename="package://waiteronix/meshes/F_W_Front_Right.STL" />
-      </geometry>
-      <material
-        name="">
-        <color
-          rgba="0.50196 0.50196 1 1" />
-      </material>
-    </visual>
-    <collision>
-      <origin
-        xyz="0 0 0"
-        rpy="0 0 0" />
-      <geometry>
-        <mesh
-          filename="package://waiteronix/meshes/F_W_Front_Right.STL" />
-      </geometry>
-    </collision>
-  </link>
-  <joint
-    name="F_W_Front_Right_Joint"
-    type="fixed">
-    <origin
-      xyz="0 0 0"
-      rpy="0 0 0" />
-    <parent
-      link="base_link" />
-    <child
-      link="F_W_Front_Right" />
-    <axis
-      xyz="0 1 0" />
-  </joint>
-  <link
-    name="F_W_Back_Left">
-    <inertial>
-      <origin
-        xyz="-0.19 0.1215 -1.622E-14"
-        rpy="0 0 0" />
-      <mass
-        value="0.059636" />
-      <inertia
-        ixx="1.6012E-05"
-        ixy="2.3169E-21"
-        ixz="-1.6362E-21"
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
Commit message: Another trial of urdf

File: waiteronix/urdf/waiteronix.xacro (robot description, xacro)
@@ -5,7 +5,4 @@
      For more information, please see http://wiki.ros.org/sw_urdf_exporter -->
   <xacro:include filename="$(find waiteronix)/urdf/waiteronix.gazebo"/>
-  <xacro:include filename="$(find waiteronix)/urdf/caster_wheels.xacro"/>
-  <xacro:include filename="$(find waiteronix)/urdf/diff_wheels.xacro"/>
-  <xacro:include filename="$(find waiteronix)/urdf/sensors.xacro"/>
   <link name="robot_footprint">
   </link>
@@ -107,3 +104,486 @@
       xyz="0 0 0" />
   </joint>
+  <link
+    name="Right_Wheel">
+    <inertial>
+      <origin
+        xyz="2.5996E-07 0.037854 6.57E-06"
+        rpy="0 0 0" />
+      <mass
+        value="1.21" />
+      <inertia
+        ixx="0.0022228"
+        ixy="-1.8762E-08"
+        ixz="1.5736E-09"
+        iyy="0.0036326"
+        iyz="-4.7418E-07"
+        izz="0.0022228" />
+    </inertial>
+    <visual>
+      <origin
+        xyz="0 0 0"
+        rpy="0 0 0" />
+      <geometry>
+        <mesh
+          filename="package://waiteronix/meshes/Right_Wheel.STL" />
+      </geometry>
+      <material
+        name="">
+        <color
+          rgba="0.75294 0.75294 0.75294 1" />
+      </material>
+    </visual>
+    <collision>
+      <origin
+        xyz="0 0 0"
+        rpy="0 0 0" />
+      <geometry>
+        <mesh
+          filename="package://waiteronix/meshes/Right_Wheel.STL" />
+      </geometry>
+    </collision>
+  </link>
+  <joint
+    name="Right_Wheel_Joint"
+    type="continuous">
+    <origin
+      xyz="-0.0087223 -0.224 0.054"
+      rpy="0 0 0" />
+    <parent
+      link="base_link" />
+    <child
+      link="Right_Wheel" />
+    <axis
+      xyz="0 -1 0" />
+    <limit
+      effort="40"
+      velocity="10" />
+  </joint>
+  <link
+    name="Left_Wheel">
+    <inertial>
+      <origin
+        xyz="2.5996E-07 -0.037854 6.57E-06"
+        rpy="0 0 0" />
+      <mass
+        value="1.21" />
+      <inertia
+        ixx="0.0022228"
+        ixy="1.8762E-08"
+        ixz="1.5736E-09"
+        iyy="0.0036326"
+        iyz="4.7418E-07"
+        izz="0.0022228" />
+    </inertial>
+    <visual>
+      <origin
+        xyz="0 0 0"
+        rpy="0 0 0" />
+      <geometry>
+        <mesh
+          filename="package://waiteronix/meshes/Left_Wheel.STL" />
+      </geometry>
+      <material
+        name="">
+        <color
+          rgba="0.75294 0.75294 0.75294 1" />
+      </material>
+    </visual>
+    <collision>
+      <origin
+        xyz="0 0 0"
+        rpy="0 0 0" />
+      <geometry>
+        <mesh
+          filename="package://waiteronix/meshes/Left_Wheel.STL" />
+      </geometry>
+    </collision>
+  </link>
+  <joint
+    name="Left_Wheel_Joint"
+    type="continuous">
+    <origin
+      xyz="-0.0087223 0.224 0.054"
+      rpy="0 0 0" />
+    <parent
+      link="base_link" />
+    <child
+      link="Left_Wheel" />
+    <axis
+      xyz="0 -1 0" />
+    <limit
+      effort="40"
+      velocity="10" />
+  </joint>
+  <link
+    name="Camera">
+    <inertial>
+      <origin
+        xyz="-0.027769 0.064365 -0.00028163"
+        rpy="0 0 0" />
+      <mass
+        value="0.55893" />
+      <inertia
+        ixx="0.0029329"
+        ixy="-9.3578E-07"
+        ixz="8.9611E-08"
+        iyy="0.00023177"
+        iyz="-9.4508E-09"
+        izz="0.0030272" />
+    </inertial>
+    <visual>
+      <origin
+        xyz="0 0 0"
+        rpy="0 0 0" />
+      <geometry>
+        <mesh
+          filename="package://waiteronix/meshes/Camera.STL" />
+      </geometry>
+      <material
+        name="">
+        <color
+          rgba="0.49412 0.49412 0.49412 1" />
+      </material>
+    </visual>
+    <collision>
+      <origin
+        xyz="0 0 0"
+        rpy="0 0 0" />
+      <geometry>
+        <mesh
+          filename="package://waiteronix/meshes/Camera.STL" />
+      </geometry>
+    </collision>
+  </link>
+  <joint
+    name="Camera_Joint"
+    type="fixed">
+    <origin
+      xyz="0.24478 -0.064307 0.0965"
+      rpy="0 0 0" />
+    <parent
+      link="base_link" />
+    <child
+      link="Camera" />
+    <axis
+      xyz="1 0 0" />
+  </joint>
+  <link
+    name="Lidar">
+    <inertial>
+      <origin
+        xyz="8.3267E-17 -1.9976E-15 -0.013917"
+        rpy="0 0 0" />
+      <mass
+        value="0.12331" />
+      <inertia
+        ixx="8.5672E-05"
+        ixy="-3.3087E-22"
+        ixz="-3.3193E-19"
+        iyy="8.5672E-05"
+        iyz="-1.4388E-23"
+        izz="0.00010203" />
+    </inertial>
+    <visual>
+      <origin
+        xyz="0 0 0"
+        rpy="0 0 0" />
+      <geometry>
+        <mesh
+          filename="package://waiteronix/meshes/Lidar.STL" />
+      </geometry>
+      <material
+        name="">
+        <color
+          rgba="0 0.75294 0 1" />
+      </material>
+    </visual>
+    <collision>
+      <origin
+        xyz="0 0 0"
+        rpy="0 0 0" />
+      <geometry>
+        <mesh
+          filename="package://waiteronix/meshes/Lidar.STL" />
+      </geometry>
+    </collision>
+  </link>
+  <joint
+    name="Lidar_Joint"
+    type="fixed">
+    <origin
+      xyz="0.185 0 0.21663"
+      rpy="0 0 0" />
+    <parent
+      link="base_link" />
+    <child
+      link="Lidar" />
+    <axis
+      xyz="0 0 1" />
+  </joint>
+  <link
+    name="IMU">
+    <inertial>
+      <origin
+        xyz="-1.8518E-16 -6.2326E-15 -0.005"
+        rpy="0 0 0" />
+      <mass
+        value="0.0007854" />
+      <inertia
+        ixx="1.1454E-08"
+        ixy="1.831E-25"
+        ixz="-3.3736E-23"
+        iyy="1.1454E-08"
+        iyz="1.7323E-23"
+        izz="9.8175E-09" />
+    </inertial>
+    <visual>
+      <origin
+        xyz="0 0 0"
+        rpy="0 0 0" />
+      <geometry>
+        <mesh
+          filename="package://waiteronix/meshes/IMU.STL" />
+      </geometry>
+      <material
+        name="">
+        <color
+          rgba="0 0.75294 0 1" />
+      </material>
+    </visual>
+    <collision>
+      <origin
+        xyz="0 0 0"
+        rpy="0 0 0" />
+      <geometry>
+        <mesh
+          filename="package://waiteronix/meshes/IMU.STL" />
+      </geometry>
+    </collision>
+  </link>
+  <joint
+    name="IMU_Joint"
+    type="fixed">
+    <origin
+      xyz="0 0 0.289"
+      rpy="0 0 0" />
+    <parent
+      link="base_link" />
+    <child
+      link="IMU" />
+    <axis
+      xyz="0 0 1" />
+  </joint>
+  <link
+    name="F_W_Front_Left">
+    <inertial>
+      <origin
+        xyz="0.13868 0.123 -1.4438E-14"
+        rpy="0 0 0" />
+      <mass
+        value="0.059636" />
+      <inertia
+        ixx="1.6012E-05"
+        ixy="-1.927E-20"
+        ixz="-9.0002E-22"
+        iyy="2.7287E-05"
+        iyz="-2.1253E-20"
+        izz="1.6012E-05" />
+    </inertial>
+    <visual>
+      <origin
+        xyz="0 0 0"
+        rpy="0 0 0" />
+      <geometry>
+        <mesh
+          filename="package://waiteronix/meshes/F_W_Front_Left.STL" />
+      </geometry>
+      <material
+        name="">
+        <color
+          rgba="0.50196 0.50196 1 1" />
+      </material>
+    </visual>
+    <collision>
+      <origin
+        xyz="0 0 0"
+        rpy="0 0 0" />
+      <geometry>
+        <mesh
+          filename="package://waiteronix/meshes/F_W_Front_Left.STL" />
+      </geometry>
+    </collision>
+  </link>
+  <joint
+    name="F_W_Front_Left_Joint"
+    type="fixed">
+    <origin
+      xyz="0 0 0"
+      rpy="0 0 0" />
+    <parent
+      link="base_link" />
+    <child
+      link="F_W_Front_Left" />
+    <axis
+      xyz="0 1 0" />
+  </joint>
+  <link
+    name="F_W_Front_Right">
+    <inertial>
+      <origin
+        xyz="0.13868 -0.123 2.4819E-14"
+        rpy="0 0 0" />
+      <mass
+        value="0.059636" />
+      <inertia
+        ixx="1.6012E-05"
+        ixy="5.4827E-21"
+        ixz="-3.2336E-22"
+        iyy="2.7287E-05"
+        iyz="-3.8765E-20"
+        izz="1.6012E-05" />
+    </inertial>
+    <visual>
+      <origin
+        xyz="0 0 0"
+        rpy="0 0 0" />
+      <geometry>
+        <mesh
+          filename="package://waiteronix/meshes/F_W_Front_Right.STL" />
+      </geometry>
+      <material
+        name="">
+        <color
+          rgba="0.50196 0.50196 1 1" />
+      </material>
+    </visual>
+    <collision>
+      <origin
+        xyz="0 0 0"
+        rpy="0 0 0" />
+      <geometry>
+        <mesh
+          filename="package://waiteronix/meshes/F_W_Front_Right.STL" />
+      </geometry>
+    </collision>
+  </link>
+  <joint
+    name="F_W_Front_Right_Joint"
+    type="fixed">
+    <origin
+      xyz="0 0 0"
+      rpy="0 0 0" />
+    <parent
+      link="base_link" />
+    <child
+      link="F_W_Front_Right" />
+    <axis
+      xyz="0 1 0" />
+  </joint>
+  <link
+    name="F_W_Back_Left">
+    <inertial>
+      <origin
+        xyz="-0.19 0.1215 -1.622E-14"
+        rpy="0 0 0" />
+      <mass
+        value="0.059636" />
+      <inertia
+        ixx="1.6012E-05"
+        ixy="2.3169E-21"
+        ixz="-1.6362E-21"
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
Commit message: chages

File: waiteronix/urdf/waiteronix.xacro (robot description, xacro)
@@ -155,5 +155,8 @@
       link="Right_Wheel" />
     <axis
-      xyz="0 1 0" />
+      xyz="0 -1 0" />
+    <limit
+      effort="40"
+      velocity="10" />
   </joint>
   <link
@@ -208,5 +211,8 @@
       link="Left_Wheel" />
     <axis
-      xyz="0 1 0" />
+      xyz="0 -1 0" />
+    <limit
+      effort="40"
+      velocity="10" />
   </joint>
   <link
@@ -373,5 +379,5 @@
     <inertial>
       <origin
-        xyz="0.13868 0.123 -1.4438E-14"
+        xyz="0.13868 0.123 0.03"
         rpy="0 0 0" />
       <mass
@@ -411,5 +417,5 @@
   <joint
     name="F_W_Front_Left_Joint"
-    type="continuous">
+    type="fixed">
     <origin
       xyz="0 0 0"
@@ -426,5 +432,5 @@
     <inertial>
       <origin
-        xyz="0.13868 -0.123 2.4819E-14"
+        xyz="0.13868 -0.123 0.03"
         rpy="0 0 0" />
       <mass
@@ -464,5 +470,5 @@
   <joint
     name="F_W_Front_Right_Joint"
-    type="continuous">
+    type="fixed">
     <origin
       xyz="0 0 0"
@@ -479,5 +485,5 @@
     <inertial>
       <origin
-        xyz="-0.19 0.1215 -1.622E-14"
+        xyz="-0.19 0.1215 0.03"
         rpy="0 0 0" />
       <mass
@@ -517,5 +523,5 @@
   <joint
     name="F_W_Back_Left_Joint"
-    type="continuous">
+    type="fixed">
     <origin
       xyz="0 0 0"
@@ -532,5 +538,5 @@
     <inertial>
       <origin
-        xyz="-0.19 -0.1215 -1.6079E-14"
+        xyz="-0.19 -0.1215 0.03"
         rpy="0 0 0" />
       <mass
@@ -570,5 +576,5 @@
   <joint
     name="F_W_Back_Right_Joint"
-    type="continuous">
+    type="fixed">
     <origin
       xyz="0 0 0"
